File: Material particulado.kicad_sch (KiCad schematic)
At the start: 0 parts

Commit message: parte analogica Keiner
Parts:
- added C1: 1uf, symbol Device:C
- added R1: 15k, symbol Device:R
- added R2, R3: 2.2k, symbol Device:R
- added R4: 1k, symbol Device:R
- added U1: ESP32-S3-WROOM-1, RF_Module:ESP32-S3-WROOM-1, symbol RF_Module:ESP32-S3-WROOM-1
- added U2: LM35-D, Package_SO:SOIC-8_3.9x4.9mm_P1.27mm, symbol Sensor_Temperature:LM35-D
- added U3, U4: LM358_DFN, Package_DFN_QFN:DFN-8-1EP_2x2mm_P0.5mm_EP1.05x1.75mm, symbol Amplifier_Operational:LM358_DFN
Connections:
- new net: R3.1, U1.2 (3V3), U2.8 (+V_{S}), U3.8 (V+), U4.8 (V+)
- new net: C1.2, R2.1, R3.2, R4.1, U3.2 (-)
- new net: C1.1, R4.2, U3.1, U4.3 (+)
- new net: R1.1, U2.4 (GND)
- new net: U1.32 (IO39), U2.1 (V_{OUT})
- new net: U4.1, U4.2 (-)
- new net GNDREF: R1.2, R2.2, U1.1 (GND), U1.40 (GND), U1.41 (GND), U3.4 (V-), U4.4 (V-)

Commit message: Editando Huellas
Parts:
- added R5: R_US, symbol Device:R_US
- added U5: (no value), 0.96huella:Sin título, symbol pantalla huella:Oled_0.96
Connections:
- net GNDREF: now also U5.1 (GND)
- net at R3.1, U1.2 (3V3), U2.8 (+V_{S})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: now also U5.2 (VCC)
- net at U1.12 (IO8): now also U5.4 (SDA)
- net at U1.17 (IO9): now also U5.3 (SCK)

Commit message: Organizando Huellas y smd -yara
Parts:
- C1: footprint (none) -> Capacitor_SMD:C_0805_2012Metric
- R1, R4: footprint (none) -> Resistor_SMD:R_0805_2012Metric_Pad1.20x1.40mm_HandSolder
- R2, R3: footprint (none) -> Resistor_SMD:R_0805_2012Metric
Changed lines of the file:
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@@
 			)
 		)
-		(property "Footprint" ""
+		(property "Footprint" "Resistor_SMD:R_0805_2012Metric"
 			(at 116.332 57.15 90)
 			(hide yes)
@@
 			)
 		)
-		(property "Footprint" ""
+		(property "Footprint" "Resistor_SMD:R_0805_2012Metric_Pad1.20x1.40mm_HandSolder"
 			(at 139.7 42.418 90)
 			(hide yes)
@@
 			)
 		)
-		(property "Footprint" ""
+		(property "Footprint" "Resistor_SMD:R_0805_2012Metric_Pad1.20x1.40mm_HandSolder"
 			(at 102.362 76.2 90)
 			(hide yes)
@@
 			)
 		)
-		(property "Footprint" ""
+		(property "Footprint" "Resistor_SMD:R_0805_2012Metric"
 			(at 116.332 76.2 90)
-			(hide yes)
 			(show_name no)
 			(do_not_autoplace no)
@@
 			)
 		)
-		(property "Footprint" ""
+		(property "Footprint" "Capacitor_SMD:C_0805_2012Metric"
 			(at 135.89 46.0248 0)
 			(hide yes)

Commit message: Corte cables
Parts:
- removed R5: R_US, symbol Device:R_US
Connections:
- net GNDREF: no longer U1.1 (GND), U1.40 (GND), U1.41 (GND), U5.1 (GND)
- net at R3.1, U2.8 (+V_{S}), U3.8 (V+)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: no longer U1.2 (3V3), U5.2 (VCC)
- new net: U1.1 (GND), U1.40 (GND), U1.41 (GND), U5.1 (GND)
- new net: U1.2 (3V3), U5.2 (VCC)
Changed lines of the file:
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@@
-	)
-	(junction
-		(at 62.23 106.68)
-		(diameter 0)
-		(color 0 0 0 0)
 	)
 	(junction
@@
 	)
 	(junction
-		(at 50.8 38.1)
-		(diameter 0)
-		(color 0 0 0 0)
-	)
-	(junction
 		(at 118.11 38.1)
 		(diameter 0)
@@
 		(color 0 0 0 0)
 	)
-	(junction
-		(at 104.14 38.1)
-		(diameter 0)
-		(color 0 0 0 0)
-	)
 	(wire
 		(pts
@@
 	(wire
 		(pts
-			(xy 50.8 36.83) (xy 50.8 38.1)
-		)
-		(stroke
-			(width 0)
-			(type default)
-		)
-	)
-	(wire
-		(pts
 			(xy 104.14 90.17) (xy 104.14 95.25)
 		)
@@
 	(wire
 		(pts
-			(xy 95.25 106.68) (xy 95.25 90.17)
+			(xy 50.8 36.83) (xy 50.8 50.8)
 		)
 		(stroke
@@
 	(wire
 		(pts
-			(xy 62.23 106.68) (xy 95.25 106.68)
-		)
-		(stroke
-			(width 0)
-			(type default)
-		)
-	)
-	(wire
-		(pts
 			(xy 104.14 38.1) (xy 104.14 48.26)
 		)
@@
 	(wire
 		(pts
-			(xy 95.25 90.17) (xy 104.14 90.17)
-		)
-		(stroke
-			(width 0)
-			(type default)
-		)
-	)
-	(wire
-		(pts
-			(xy 50.8 38.1) (xy 104.14 38.1)
-		)
-		(stroke
-			(width 0)
-			(type default)
-		)
-	)
-	(wire
-		(pts
 			(xy 104.14 90.17) (xy 118.11 90.17)
 		)
@@
 		(pts
 			(xy 135.89 71.12) (xy 135.89 90.17)
-		)
-		(stroke
-			(width 0)
-			(type default)
-		)
-	)
-	(wire
-		(pts
-			(xy 50.8 38.1) (xy 50.8 50.8)
 		)
 		(stroke
@@
 					(unit 1)
 				)
-			)
-		)
-	)
-	(symbol
-		(lib_id "Device:R_US")
-		(at 163.83 91.44 0)
-		(unit 1)
-		(body_style 1)
-		(exclude_from_sim no)
-		(in_bom yes)
-		(on_board yes)
-		(in_pos_files yes)
-		(dnp no)
-		(fields_autoplaced yes)
-		(property "Reference" "R5"
-			(at 166.37 90.1699 0)
-			(show_name no)
-			(do_not_autoplace no)
-			(effects
-				(font
-					(size 1.27 1.27)
-				)
-				(justify left)
-			)
-		)
-		(property "Value" "R_US"
-			(at 166.37 92.7099 0)
-			(show_name no)
-			(do_not_autoplace no)
-			(effects
-				(font
-					(size 1.27 1.27)
-				)
-				(justify left)
-			)
-		)
-		(property "Footprint" ""
-			(at 164.846 91.694 90)
-			(hide yes)
-			(show_name no)
-			(do_not_autoplace no)
-			(effects
-				(font
-					(size 1.27 1.27)
-				)
-			)
-		)
-		(property "Datasheet" ""
-			(at 163.83 91.44 0)
-			(hide yes)
-			(show_name no)
-			(do_not_autoplace no)
-			(effects
-				(font
-					(size 1.27 1.27)
-				)
-			)
-		)
-		(property "Description" "Resistor, US symbol"
-			(at 163.83 91.44 0)
-			(hide yes)
-			(show_name no)
-			(do_not_autoplace no)
-			(effects
-				(font
-					(size 1.27 1.27)
-				)
-			)
-		)
-		(pin "2"
-		)
-		(pin "1"
-		)
-		(instances
-			(project "Material particulado"
-				(path "/afc7c7c8-0489-473c-810c-6c8b74730196"
-					(reference "R5")
-					(unit 1)
-				)

Commit message: Puse etiquetas y corte cables
Parts:
- removed C1: 1uf, Capacitor_SMD:C_0805_2012Metric, symbol Device:C
- removed R3: 2.2k, Resistor_SMD:R_0805_2012Metric, symbol Device:R
- removed R4: 1k, Resistor_SMD:R_0805_2012Metric_Pad1.20x1.40mm_HandSolder, symbol Device:R
- removed U4: LM358_DFN, Package_DFN_QFN:DFN-8-1EP_2x2mm_P0.5mm_EP1.05x1.75mm, symbol Amplifier_Operational:LM358_DFN
Connections:
- net GNDREF is gone; now on net GND: R1.2, R2.2, U3.4 (V-)
- net +5V: now reaches U2.8 (+V_{S}), U3.8 (V+)
- net Salida: now reaches U3.1
- net GND: now reaches U1.1 (GND), U1.40 (GND), U1.41 (GND), U5.1 (GND)
- net +3V3: now reaches U1.2 (3V3), U5.2 (VCC)
- net 17(I09): now reaches U5.3 (SCK)
- net 17(I09): no longer U1.17 (IO9)
- net 12(I08): now reaches U5.4 (SDA)
- net 12(I08): no longer U1.12 (IO8)
- net 32(I039): now reaches U2.1 (V_{OUT})
- net 32(I039): no longer U1.32 (IO39)
- new net SCK: U1.17 (IO9)
- new net SDA: U1.12 (IO8)
- new net Vout(LM35): U1.32 (IO39)
Other:
- moved on the sheet: R1, R2

Commit message: agregue el usb, un regulador de 5v a 3.3v y el bloque pms
Parts:
- added J1: pms, symbol Connector:Screw_Terminal_01x06
- added P1: USB_C_Plug_USB2.0, symbol Connector:USB_C_Plug_USB2.0
- added U4: Regulador de 5v a 3.3v, Package_TO_SOT_SMD:SOT-223-3_TabPin2, symbol Regulator_Linear:AMS1117-3.3
Connections:
- net +3V3: now also U4.2 (VO)
- net +5V: now also P1.A4 (VBUS), P1.A9 (VBUS), P1.B4 (VBUS), P1.B9 (VBUS), U4.3 (VI)
- net GND: now also P1.A1 (GND), P1.A12 (GND), P1.B1 (GND), P1.B12 (GND), U4.1 (GND)

Commit message: Hice cambios en las huellas
Parts:
- removed J1: pms, symbol Connector:Screw_Terminal_01x06
- added J1: PMS, TerminalBlock_Phoenix:TerminalBlock_Phoenix_PTSM-0,5-4-2,5-V-SMD_1x04-1MP_P2.50mm_Vertical, symbol Connector:Screw_Terminal_01x04
- Oled1: renamed from U5; footprint 0.96huella:Sin título -> TerminalBlock_Phoenix:TerminalBlock_Phoenix_PTSM-0,5-4-2,5-V-SMD_1x04-1MP_P2.50mm_Vertical
- P1: footprint (none) -> Connector_USB:USB_C_Plug_ShenzhenJingTuoJin_918-118A2021Y40002_Vertical
Connections:
- net +5V: now also J1.1 (Pin_1)
- net GND: now also J1.2 (Pin_2)
- net TX(PMS): now reaches U1.36 (RXD0)
- net RX(PMS): now reaches U1.37 (TXD0)
- new net RX(D0): J1.4 (Pin_4)
- new net TX(D0): J1.3 (Pin_3)

Commit message: cambie pistas-yara
Changed lines of the file:
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@@
+	(wire
+		(pts
+			(xy 71.12 55.88) (xy 66.04 55.88)
+		)
+		(stroke
+			(width 0)
+			(type default)
+		)
+	)
 	(wire
 		(pts
@@
 	(wire
 		(pts
+			(xy 68.58 63.5) (xy 68.58 58.42)
+		)
+		(stroke
+			(width 0)
+			(type default)
+		)
+	)
+	(wire
+		(pts
 			(xy 129.54 67.31) (xy 129.54 68.58)
 		)
@@
 	(wire
 		(pts
+			(xy 71.12 54.61) (xy 71.12 55.88)
+		)
+		(stroke
+			(width 0)
+			(type default)
+		)
+	)
+	(wire
+		(pts
 			(xy 24.13 29.21) (xy 24.13 31.75)
 		)
@@
 	(wire
 		(pts
-			(xy 66.04 58.42) (xy 68.58 58.42)
+			(xy 68.58 63.5) (xy 90.17 63.5)
 		)
 		(stroke
@@
 	(wire
 		(pts
-			(xy 133.35 30.48) (xy 129.54 30.48)
-		)
-		(stroke
-			(width 0)
-			(type default)
-		)
-	)
-	(wire
-		(pts
 			(xy 135.89 71.12) (xy 135.89 74.93)
 		)
@@
 	(wire
 		(pts
+			(xy 128.27 30.48) (xy 133.35 30.48)
+		)
+		(stroke
+			(width 0)
+			(type default)
+		)
+	)
+	(wire
+		(pts
 			(xy 66.04 83.82) (xy 71.12 83.82)
 		)
@@
 	(wire
 		(pts
-			(xy 129.54 33.02) (xy 133.35 33.02)
+			(xy 127 33.02) (xy 133.35 33.02)
 		)
 		(stroke
@@
 	(wire
 		(pts
-			(xy 66.04 55.88) (xy 68.58 55.88)
+			(xy 71.12 54.61) (xy 72.39 54.61)
 		)
 		(stroke
@@
 	(wire
 		(pts
+			(xy 68.58 58.42) (xy 66.04 58.42)
+		)
+		(stroke
+			(width 0)
+			(type default)
+		)
+	)
+	(wire
+		(pts
 			(xy 69.85 30.48) (xy 73.66 30.48)
 		)
@@
 	(global_label "TX(D0)"
 		(shape input)
-		(at 129.54 30.48 180)
+		(at 128.27 30.48 180)
 		(fields_autoplaced yes)
 		(effects
@@
 		)
 		(property "Intersheetrefs" "${INTERSHEET_REFS}"
-			(at 120.2048 30.48 0)
+			(at 118.9348 30.48 0)
 			(hide yes)
 			(show_name no)
@@
 	(global_label "TX(PMS)"
 		(shape input)
-		(at 68.58 58.42 0)
+		(at 90.17 63.5 0)
 		(fields_autoplaced yes)
 		(effects
@@
 		)
 		(property "Intersheetrefs" "${INTERSHEET_REFS}"
-			(at 79.3666 58.42 0)
+			(at 100.9566 63.5 0)
 			(hide yes)
 			(show_name no)
@@
 	(global_label "RX(PMS)"
 		(shape input)
-		(at 68.58 55.88 0)
+		(at 72.39 54.61 0)
 		(fields_autoplaced yes)
 		(effects
@@
 		)
 		(property "Intersheetrefs" "${INTERSHEET_REFS}"
-			(at 79.669 55.88 0)
+			(at 83.479 54.61 0)
 			(hide yes)
 			(show_name no)
@@
 	(global_label "RX(D0)"
 		(shape input)
-		(at 129.54 33.02 180)
+		(at 127 33.02 180)
 		(fields_autoplaced yes)
 		(effects
@@
 		)
 		(property "Intersheetrefs" "${INTERSHEET_REFS}"
-			(at 119.9024 33.02 0)
-			(hide yes)
-			(show_name no)
+			(at 117.3624 33.02 0)
+			(hide yes)
+			(show_name no)
